File: AJH_Wasp/AJH_Wasp_1_02.brd (EAGLE design)
At the start: 19 x 108.4 mm, 71 parts, among them IC1 LM1117-5.0, IC2 4069D, IC3 LM13700M, IC4 TL072D, J100 PJ301_THONKICONN8, J101 PJ301_THONKICONN8, J102 PJ301_THONKICONN6, SW1 submini-2T

Commit message: Wasp update v1.02 - correct reversed Q pot
Parts:
- moved R5 0.58 mm to (16.4, 81.7)
- moved C6 0.56 mm to (16.4, 86.0)
- moved R3 0.56 mm to (16.4, 88.0)
- moved R4 0.56 mm to (16.4, 83.9)
- moved D5 0.24 mm to (4.13, 81.7)
- moved D6 0.16 mm to (4.21, 80.8)
- moved R7 0.16 mm to (16.8, 79.1)
- moved R13 0.08 mm to (6.03, 74.5)
Connections:
- net BP: now also R101.P$3; no longer R101.P$1
- net N$12: now also R101.P$1; no longer R101.P$3
Routing:
- net BP: track 58.1 -> 77.0 mm, vias 2 -> 1
- net N$12: track 14.0 -> 10.1 mm, vias 1 -> 0
- net HP: track 71.7 -> 74.8 mm
- net N$19: track 27.7 -> 29.3 mm
- net N$16: track 28.8 -> 29.4 mm
- net NP: track 66.3 -> 66.9 mm
Other:
- board text added: "Wasp v1.02, copyright forestcaver, 2020"
- board text removed: "Wasp v1.0, copyright forestcaver, 2020"
