File: AJH_SSI2144/AJH_ss12144_v1_01.brd (EAGLE design)
At the start: 19 x 106.8 mm, 56 parts, among them IC1 LM4040 5.0V, IC2 TL074D, IC3 TL072D, J100 PJ301_THONKICONN6, J101 PJ301_THONKICONN6, J102 PJ301_THONKICONN6, J103 PJ301_THONKICONN6, U1 BCM847BS

Commit message: AJH_ssi2144 corrections to prototype
Parts:
- added C16: 3.3n, rcl:C0603
- R11: value 50k -> 100k
- R9: value 200k -> 100k
- moved R19 2.03 mm to (3.68, 38.9)
- moved C10 1.02 mm to (3.68, 36.8)
- moved U1 0.52 mm to (3.43, 34.2)
- moved C13 0.13 mm to (3.68, 31.4)
Connections:
- net -10V: now also R100.P$3
- net -5V: no longer R4.1
- net 10V: now also R4.1
- net GND: no longer R100.P$3
- net N$24: now also C16.1
- net N$28: now also C16.2
Routing:
- net -10V: track 11.1 -> 24.3 mm
- net N$28: track 24.9 -> 31.9 mm
- net 10V: track 40.0 -> 42.6 mm
- net N$3: track 44.6 -> 42.1 mm
- net -5V: track 6.00 -> 3.86 mm
- net N$9: track 6.97 -> 6.16 mm
- net N$24: track 8.01 -> 8.71 mm
- net N$16: track 9.65 -> 8.99 mm
- net N$7: track 82.1 -> 81.6 mm, vias 2 -> 3
Other:
- board text added: "ssi2144 lpf v1.01, copyright forestcaver 2020"
- board text removed: "ssi2144 lpf v1.0, copyright forestcaver 2020"
