File: AJH_SSI2144/AJH_ss12144_v1_01.sch (EAGLE design)
At the start: 56 parts, among them IC1 LM4040 5.0V, IC2 TL074D, IC3 TL072D, J100 PJ301_THONKICONN6, J101 PJ301_THONKICONN6, J102 PJ301_THONKICONN6, J103 PJ301_THONKICONN6, U1 BCM847BS

Commit message: AJH_ssi2144 corrections to prototype
Parts:
- added C16: 3.3n, rcl:C-USC0603
- R11: value 50k -> 100k
- R9: value 200k -> 100k
Connections:
- net -10V: now also R100.A
- net -5V: no longer R4.1
- net 10V: now also R4.1
- net GND: no longer R100.A
- net N$24: now also C16.1
- net N$28: now also C16.2
Other:
- note added: "SSI2144 needs ~ -19mv/oct, but parts have quite wide variability So probably best for R11 to be 100k, or use 50k and adjust the 162k to suit"
- moved on the sheet: R100, R19, R2, R24, R25
