File: AJH_SSI2144/AJH_ss12144_v1_02.sch (EAGLE design)
At the start: 57 parts, among them IC1 LM4040 5.0V, IC2 TL074D, IC3 TL072D, J100 PJ301_THONKICONN6, J101 PJ301_THONKICONN6, J102 PJ301_THONKICONN6, J103 PJ301_THONKICONN6, U1 BCM847BS

Commit message: Add 2B_VCA, add some comments on ssi2144 schematic
Parts:
- R16: value 162k -> 130k
Other:
- note added: "R21 and R11 are optional - the trimmer can be used to set the offset of the frequency pot."
- note added: "SSI2144 needs ~ -19mv/oct, but parts have quite wide variability So choose either R11=100k and R16=130k; or R11=50k and R16=162k"
- note removed: "SSI2144 needs ~ -19mv/oct, but parts have quite wide variability So probably best for R11 to be 100k, or use 50k and adjust the 162k to suit"
Changed lines of the file:
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@@
 <part name="GND1" library="SparkFun" deviceset="GND" device=""/>
 <part name="R2" library="resistor" deviceset="R-US_" device="R0603" value="100k"/>
-<part name="R16" library="resistor" deviceset="R-US_" device="R0603" value="162k"/>
+<part name="R16" library="resistor" deviceset="R-US_" device="R0603" value="130k"/>
 <part name="R17" library="resistor" deviceset="R-US_" device="R0603" value="100k"/>
 <part name="R23" library="resistor" deviceset="R-US_" device="R0603" value="100k"/>
@@
 <text x="-109.22" y="-60.96" size="1.778" layer="91">667-ERA-V33J102V - obsolete
 667-ERT-J1VK102FM - check datasheet</text>
-<text x="-152.4" y="-2.54" size="1.778" layer="91">SSI2144 needs ~ -19mv/oct, but parts have quite wide variability
-So probably best for R11 to be 100k, or use 50k and adjust the 162k to suit</text>
+<text x="-142.24" y="-2.54" size="1.778" layer="91">SSI2144 needs ~ -19mv/oct, but parts have quite wide variability
+So choose either R11=100k and R16=130k; or  R11=50k and R16=162k</text>
+<text x="-53.34" y="-40.64" size="1.778" layer="91">R21 and R11 are optional - the trimmer can
+be used to set the offset of the frequency pot.</text>
 </plain>
 <instances>
