File: AJH_100_ADSR/AJH_100m_ADSR_1_01.sch (EAGLE design)
At the start: 66 parts, among them IC1 TL072D, IC2 TL072D, J100 PJ301_THONKICONN6, J101 PJ301_THONKICONN6, J102 PJ301_THONKICONN6, Q1 MMBT3904, Q10 MMBT3904, Q2 MMBT3906, Q3 MMBT3906, Q4 MMBT3904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

Commit message: Updated a100  adsr with correct pot direction
Connections:
- removed net N$36: D3.C, R100.E
- removed net N$56: R101.E, R6.1
- removed net N$60: R103.E, R22.1
- new net N$5: D3.C, R100.A
- new net N$7: R101.A, R6.1
- new net N$8: R103.A, R22.1
- net N$38: now also R100.E, R101.E, R103.E; no longer R100.A, R101.A, R103.A
Changed lines of the file:
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@@
 <?xml version="1.0" encoding="utf-8"?>
 <!DOCTYPE eagle SYSTEM "eagle.dtd">
-<eagle version="9.5.2">
+<eagle version="9.6.2">
 <drawing>
 <settings>
@@
 <attribute name="VALUE" x="-54.61" y="0.762" size="1.778" layer="96" rot="R180"/>
 </instance>
-<instance part="R100" gate="G$1" x="-43.18" y="48.26" smashed="yes" rot="R90">
-<attribute name="NAME" x="-40.64" y="43.18" size="1.778" layer="95" rot="R180"/>
-<attribute name="VALUE" x="-40.64" y="45.72" size="1.778" layer="96" rot="R180"/>
-</instance>
-<instance part="R101" gate="G$1" x="-43.18" y="-2.54" smashed="yes" rot="R90">
-<attribute name="NAME" x="-40.64" y="-7.62" size="1.778" layer="95" rot="R180"/>
-<attribute name="VALUE" x="-40.64" y="-5.08" size="1.778" layer="96" rot="R180"/>
-</instance>
-<instance part="R103" gate="G$1" x="-43.18" y="-55.88" smashed="yes" rot="R90">
-<attribute name="NAME" x="-40.64" y="-60.96" size="1.778" layer="95" rot="R180"/>
-<attribute name="VALUE" x="-40.64" y="-58.42" size="1.778" layer="96" rot="R180"/>
+<instance part="R100" gate="G$1" x="-43.18" y="48.26" smashed="yes" rot="MR90">
+<attribute name="NAME" x="-45.72" y="43.18" size="1.778" layer="95" rot="MR180"/>
+<attribute name="VALUE" x="-45.72" y="45.72" size="1.778" layer="96" rot="MR180"/>
+</instance>
+<instance part="R101" gate="G$1" x="-43.18" y="-2.54" smashed="yes" rot="MR90">
+<attribute name="NAME" x="-45.72" y="-7.62" size="1.778" layer="95" rot="MR180"/>
+<attribute name="VALUE" x="-45.72" y="-5.08" size="1.778" layer="96" rot="MR180"/>
+</instance>
+<instance part="R103" gate="G$1" x="-43.18" y="-55.88" smashed="yes" rot="MR90">
+<attribute name="NAME" x="-45.72" y="-60.96" size="1.778" layer="95" rot="MR180"/>
+<attribute name="VALUE" x="-45.72" y="-58.42" size="1.778" layer="96" rot="MR180"/>
 </instance>
 <instance part="Q7" gate="G$1" x="-124.46" y="-68.58" smashed="yes">
@@
 </segment>
 </net>
-<net name="N$36" class="0">
-<segment>
-<pinref part="D3" gate="G$1" pin="C"/>
-<wire x1="-81.28" y1="48.26" x2="-50.8" y2="48.26" width="0.1524" layer="91"/>
-<pinref part="R100" gate="G$1" pin="E"/>
-</segment>
-</net>
 <net name="N$38" class="0">
 <segment>
-<pinref part="R100" gate="G$1" pin="S"/>
-<wire x1="-43.18" y1="53.34" x2="-43.18" y2="55.88" width="0.1524" layer="91"/>
 <wire x1="-43.18" y1="55.88" x2="-33.02" y2="55.88" width="0.1524" layer="91"/>
-<wire x1="-33.02" y1="55.88" x2="-33.02" y2="48.26" width="0.1524" layer="91"/>
-<pinref part="R100" gate="G$1" pin="A"/>
-<wire x1="-33.02" y1="48.26" x2="-35.56" y2="48.26" width="0.1524" layer="91"/>
 <wire x1="-33.02" y1="55.88" x2="-33.02" y2="60.96" width="0.1524" layer="91"/>
 <junction x="-33.02" y="55.88"/>
+<wire x1="-33.02" y1="55.88" x2="-33.02" y2="48.26" width="0.1524" layer="91"/>
 <wire x1="-33.02" y1="48.26" x2="-33.02" y2="5.08" width="0.1524" layer="91"/>
-<junction x="-33.02" y="48.26"/>
-<pinref part="R101" gate="G$1" pin="S"/>
-<wire x1="-43.18" y1="2.54" x2="-43.18" y2="5.08" width="0.1524" layer="91"/>
 <wire x1="-43.18" y1="5.08" x2="-33.02" y2="5.08" width="0.1524" layer="91"/>
-<wire x1="-33.02" y1="5.08" x2="-33.02" y2="-2.54" width="0.1524" layer="91"/>
 <junction x="-33.02" y="5.08"/>
-<pinref part="R101" gate="G$1" pin="A"/>
-<wire x1="-33.02" y1="-2.54" x2="-35.56" y2="-2.54" width="0.1524" layer="91"/>
-<pinref part="R103" gate="G$1" pin="S"/>
-<wire x1="-43.18" y1="-50.8" x2="-43.18" y2="-48.26" width="0.1524" layer="91"/>
 <wire x1="-43.18" y1="-48.26" x2="-33.02" y2="-48.26" width="0.1524" layer="91"/>
 <wire x1="-33.02" y1="-48.26" x2="-33.02" y2="-2.54" width="0.1524" layer="91"/>
-<junction x="-33.02" y="-2.54"/>
+<wire x1="-33.02" y1="-2.54" x2="-33.02" y2="5.08" width="0.1524" layer="91"/>
 <wire x1="-33.02" y1="-48.26" x2="-33.02" y2="-55.88" width="0.1524" layer="91"/>
 <junction x="-33.02" y="-48.26"/>
-<pinref part="R103" gate="G$1" pin="A"/>
-<wire x1="-33.02" y1="-55.88" x2="-35.56" y2="-55.88" width="0.1524" layer="91"/>
 <pinref part="IC2" gate="A" pin="+IN"/>
 <wire x1="-33.02" y1="60.96" x2="-25.4" y2="60.96" width="0.1524" layer="91"/>
@@
 <wire x1="-25.4" y1="25.4" x2="-25.4" y2="35.56" width="0.1524" layer="91"/>
 <junction x="-25.4" y="35.56"/>
-</segment>
-</net>
-<net name="N$56" class="0">
-<segment>
+<pinref part="R100" gate="G$1" pin="S"/>
+<wire x1="-43.18" y1="53.34" x2="-43.18" y2="55.88" width="0.1524" layer="91"/>
+<pinref part="R100" gate="G$1" pin="E"/>
+<wire x1="-35.56" y1="48.26" x2="-33.02" y2="48.26" width="0.1524" layer="91"/>
+<junction x="-33.02" y="48.26"/>
 <pinref part="R101" gate="G$1" pin="E"/>
-<pinref part="R6" gate="G$1" pin="1"/>
-<wire x1="-50.8" y1="-2.54" x2="-53.34" y2="-2.54" width="0.1524" layer="91"/>
+<wire x1="-35.56" y1="-2.54" x2="-33.02" y2="-2.54" width="0.1524" layer="91"/>
+<junction x="-33.02" y="-2.54"/>
+<pinref part="R101" gate="G$1" pin="S"/>
+<wire x1="-43.18" y1="2.54" x2="-43.18" y2="5.08" width="0.1524" layer="91"/>
+<pinref part="R103" gate="G$1" pin="S"/>
+<wire x1="-43.18" y1="-50.8" x2="-43.18" y2="-48.26" width="0.1524" layer="91"/>
+<pinref part="R103" gate="G$1" pin="E"/>
+<wire x1="-35.56" y1="-55.88" x2="-33.02" y2="-55.88" width="0.1524" layer="91"/>
 </segment>
 </net>
@@
 <pinref part="Q7" gate="G$1" pin="B"/>
 <wire x1="-142.24" y1="-68.58" x2="-127" y2="-68.58" width="0.1524" layer="91"/>
-</segment>
-</net>
-<net name="N$60" class="0">
-<segment>
-<pinref part="R22" gate="G$1" pin="1"/>
-<pinref part="R103" gate="G$1" pin="E"/>
-<wire x1="-58.42" y1="-55.88" x2="-50.8" y2="-55.88" width="0.1524" layer="91"/>
 </segment>
 </net>
@@
 </segment>
 </net>
+<net name="N$5" class="0">
+<segment>
+<pinref part="D3" gate="G$1" pin="C"/>
+<pinref part="R100" gate="G$1" pin="A"/>
+<wire x1="-81.28" y1="48.26" x2="-50.8" y2="48.26" width="0.1524" layer="91"/>
+</segment>
+</net>
+<net name="N$7" class="0">
+<segment>
+<pinref part="R101" gate="G$1" pin="A"/>
+<pinref part="R6" gate="G$1" pin="1"/>
+<wire x1="-50.8" y1="-2.54" x2="-53.34" y2="-2.54" width="0.1524" layer="91"/>
+</segment>
+</net>
+<net name="N$8" class="0">
+<segment>
+<pinref part="R22" gate="G$1" pin="1"/>
+<pinref part="R103" gate="G$1" pin="A"/>
+<wire x1="-58.42" y1="-55.88" x2="-50.8" y2="-55.88" width="0.1524" layer="91"/>
+</segment>
+</net>
