File: AJH_module_tester/AJH_module_tester-v1_00.brd (EAGLE design)
At the start: 78.9 x 106.8 mm, 133 parts, among them IC1 LM4040 4.1V, IC10 TL074D, IC2 TL074D, IC3 MCP4822SO08, IC4 LM4040DIM3-5.0V, IC5 74HC595D, IC6 74HC165N, IC7 MCP6002, IC8 LM1117-5.0, IC9 ATMEGA644A, J1 PJ301_THONKICONN6, J10 PJ301_THONKICONN6, J11 PJ301_THONKICONN6, J2 PJ301_THONKICONN6, J3 PJ301_THONKICONN6, J4 PJ301_THONKICONN6, J5 PJ301_THONKICONN6, J6 PJ301_THONKICONN6, J7 M05X2PTH, J8 PJ301_THONKICONN6, J9 PJ301_THONKICONN6, Q1 MMBT3904, Q2 20MHz, SW1 Encoder, U1 ISP

Commit message: Update module tester
Parts:
- removed C1, C15, C20, C3: 100n, rcl:C0603
- removed C10, C12: 10u, rcl:PANASONIC_A
- removed C24, C6: 4.7u, rcl:PANASONIC_A
- removed C26: 22u, rcl:PANASONIC_C
- removed C9: 100u, rcl:PANASONIC_A
- removed D3: 1N5819HW, diode:SOD123
- removed IC1: LM4040 4.1V, texas:DBZ_R-PDSO-G3
- removed IC4: LM4040DIM3-5.0V, texas:DBZ_R-PDSO-G3
- removed J11: PJ301_THONKICONN6, og-pj301:WQP_PJ_301M6
- removed R1: 10k, resistor:R0603
- removed R2: 470, resistor:R0603
- removed R29, R47, R57: 100k, rcl:R0603
- removed R48, R49, R50, R51: 51, rcl:R0603
- removed R5: 10k, rcl:R0603
- added C100, C109: 10u, rcl:PANASONIC_B
- added C101: 22u, rcl:PANASONIC_C
- added C103: 100u, rcl:PANASONIC_C
- added C105, C106, C108, C112: 100n, rcl:C0603
- added C107, C128: 4.7u, rcl:PANASONIC_B
- added D101: 1N5819HW, diode:SOD123
- added IC101: LM4040DIM3-5.0V, texas:DBZ_R-PDSO-G3
- added IC103: LM4040 4.1V, texas:DBZ_R-PDSO-G3
- added J100: M05X2PTH, og-header:AVR_ICSP
- added R104: 10k, resistor:R0603
- added R106: 470, resistor:R0603
- added R117: 10k, rcl:R0603
- added R138, R139, R140, R141, R142, R143, R144, R145: 0R, rcl:R0603
- added R146, R148, R149, R151: 51, rcl:R0603
- added R147, R150, R152: 100k, rcl:R0603
- J7: value M05X2PTH -> PJ301_THONKICONN6; device og-header:AVR_ICSP -> og-pj301:WQP_PJ_301M6
- moved J7 69.1 mm to (33.2, 30.5), flipped to the top
- moved J5 51.2 mm to (7.62, 30.5)
- moved J2 19.8 mm to (33.4, 45.5)
- moved J9 19.7 mm to (58.8, 30.5)
- moved J3 19.7 mm to (46.0, 45.5)
- moved J8 19.6 mm to (46.0, 30.5)
- moved J1 19.6 mm to (20.2, 45.5)
- moved J4 19.6 mm to (58.6, 45.5)
- moved J6 15.0 mm to (20.4, 30.5)
- renumbered C11 to C113, C13 to C116, C14 to C111, C16 to C115, C17 to C126, C18 to C114, C19 to C102, C2 to C110, C21 to C127, C22 to C121, C23 to C120, C25 to C124, C27 to C104, C28 to C122, C29 to C117, C4 to C123, C5 to C118, C7 to C125, C8 to C119, D1 to D102, D2 to D100, IC10 to IC106, IC2 to IC107, IC3 to IC102, IC5 to IC109, IC6 to IC104, IC7 to IC108, IC8 to IC100, IC9 to IC105, OK1 to OK100, Q1 to Q101, Q2 to Q100, R10 to R111, R11 to R129, R12 to R113, R13 to R107, R14 to R123, R15 to R126, R16 to R112, R17 to R156, R18 to R155, R19 to R158, R20 to R161, R21 to R160, R22 to R162, R23 to R159, R24 to R157, R25 to R153, R26 to R105, R27 to R154, R28 to R119, R3 to R137, R30 to R120, R31 to R132, R32 to R122, R33 to R131, R34 to R115, R35 to R127, R36 to R167, R37 to R166, R38 to R165, R39 to R168, R4 to R124, R40 to R164, R41 to R163, R42 to R102, R43 to R103, R44 to R128, R45 to R130, R46 to R114, R52 to R116, R53 to R121, R54 to R134, R55 to R133, R56 to R109, R58 to R118, R59 to R125, R6 to R110, R60 to R100, R61 to R101, R7 to R136, R8 to R135, R9 to R108, U1 to U100
Connections:
- new net N$61: R136.3, R142.2
- new net N$62: R136.1, R143.2
- new net N$63: R135.3, R140.2
- new net N$65: R135.1, R141.2
- new net N$67: R134.3, R139.2
- new net N$68: R134.1, R138.2
- new net N$69: R133.3, R144.2
- new net N$70: R133.1, R145.2
- net +5V: now also C101.+, C103.+, C106.1, R117.2; no longer C15.1, C26.+, C9.+, R5.2
- net -5V_ACCURATE: now also R139.1, R140.1, R142.1, R144.1; no longer R133.3, R134.3, R135.3, R136.3
- net 5V_ACCURATE: now also R138.1, R141.1, R143.1, R145.1; no longer R133.1, R134.1, R135.1, R136.1
- net DAC_TONE: now also C107.+; no longer C6.+
- net GND: now also C100.-, C101.-, C103.-, C105.2, C106.2, C108.2, C109.+, C112.2, IC101.1, IC103.1, J100.3, J100.4, J100.5, J100.6, J100.7, J100.8, J7.P1; no longer C1.2, C10.+, C12.-, C15.2, C20.2, C26.-, C3.2, C9.-, IC1.1, IC4.1, J11.P1, J7.3, J7.4, J7.5, J7.6, J7.7, J7.8
- net MIDI_IN: now also R117.1; no longer R5.1
- net N$11: now also J5.P3; no longer J1.P3
- net N$14: now also J6.P3; no longer J2.P3
- net N$16: now also J2.P3, R151.2; no longer J8.P3, R49.2
- net N$17: now also C107.-; no longer C6.-
- net N$18: now also J1.P3, R148.2; no longer J6.P3, R48.2
- net N$26: now also J7.P3; no longer J3.P3
- net N$38: now also R152.2; no longer R29.2
- net N$39: now also R147.2, R151.1; no longer R47.2, R49.1
- net N$40: now also C128.-, R152.1; no longer C24.-, R29.1
- net N$41: now also R149.1; no longer R50.1
- net N$47: now also R148.1; no longer R48.1
- net N$48: now also R147.1, R150.2; no longer R47.1, R57.2
- net N$53: now also J3.P3, R149.2; no longer J9.P3, R50.2
- net N$54: now also J4.P3, R146.2; no longer J11.P3, R51.2
- net N$55: now also R146.1; no longer R51.1
- net N$56: now also J100.1, J100.2; no longer J7.1, J7.2
- net N$57: now also R150.1; no longer R57.1
- net N$6: now also C128.+, J9.P3; no longer C24.+, J5.P3
- net N$64: now also D101.C, J100.10, J100.9; no longer D3.C, J7.10, J7.9
- net REF_-4.096: now also C108.1, IC103.2, R106.2; no longer C3.1, IC1.2, R2.2
- net REF_-5V: now also C105.1, IC101.2, R104.2; no longer C1.1, IC4.2, R1.2
- net RESET: now also C112.1; no longer C20.1
- net TONE_OUT: now also J8.P3; no longer J4.P3
- net VCC: now also C100.+; no longer C12.+
- net VEE: now also C109.-, D101.A, R104.1, R106.1; no longer C10.-, D3.A, R1.1, R2.1
Routing:
- net 5V_ACCURATE: track 53.5 -> 69.0 mm, vias 2 -> 5
- net +5V: track 389.0 -> 404.5 mm
- net -5V_ACCURATE: track 52.0 -> 63.4 mm, vias 0 -> 5
- net N$62: track 0.00 -> 4.97 mm
- net N$61: track 0.00 -> 4.69 mm
- net N$55: track 25.9 -> 30.4 mm
- net N$63: track 0.00 -> 4.35 mm
- net N$70: track 0.00 -> 4.30 mm
- net N$69: track 0.00 -> 4.23 mm
- net N$65: track 0.00 -> 4.13 mm
- net N$67: track 0.00 -> 4.03 mm
- net N$68: track 0.00 -> 3.95 mm
- net N$47: track 21.2 -> 24.7 mm
- net N$52: track 24.6 -> 21.3 mm
- net N$39: track 23.8 -> 26.9 mm
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Other:
- board text added: "Module Tester v1.00, copyright forestcaver 2020, original design Emilie Gillet"
- board text added: "Red Stripe"
