File: AJH_module_tester/AJH_module_tester-v1_00.sch (EAGLE design)
At the start: 133 parts, among them IC1 LM4040 4.1V, IC10 TL074D, IC2 TL074D, IC3 MCP4822SO08, IC4 LM4040DIM3-5.0V, IC5 74HC595D, IC6 74HC165N, IC7 MCP6002, IC8 LM1117-5.0, IC9 ATMEGA644A, J1 PJ301_THONKICONN6, J10 PJ301_THONKICONN6, J11 PJ301_THONKICONN6, J2 PJ301_THONKICONN6, J3 PJ301_THONKICONN6, J4 PJ301_THONKICONN6, J5 PJ301_THONKICONN6, J6 PJ301_THONKICONN6, J7 M05X2PTH, J8 PJ301_THONKICONN6, J9 PJ301_THONKICONN6, Q1 MMBT3904, Q2 20MHz, SW1 Encoder, U1 ISP

Commit message: Update module tester
Parts:
- removed C10, C12: 10u, rcl:CPOL-USA
- removed C24, C6: 4.7u, rcl:CPOL-USA
- removed C9: 100u, rcl:CPOL-USA
- removed J11: PJ301_THONKICONN6, og-pj301:PJ301_THONKICONN6
- added C100, C109: 10u, rcl:CPOL-USB
- added C103: 100u, rcl:CPOL-USC
- added C107, C128: 4.7u, rcl:CPOL-USB
- added J100: M05X2PTH, og-header:M05X2PTH
- added R138, R139, R140, R141, R142, R143, R144, R145: 0R, rcl:R-US_R0603
- J7: value M05X2PTH -> PJ301_THONKICONN6; device og-header:M05X2PTH -> og-pj301:PJ301_THONKICONN6
- renumbered C1 to C105, C11 to C113, C13 to C116, C14 to C111, C15 to C106, C16 to C115, C17 to C126, C18 to C114, C19 to C102, C2 to C110, C20 to C112, C21 to C127, C22 to C121, C23 to C120, C25 to C124, C26 to C101, C27 to C104, C28 to C122, C29 to C117, C3 to C108, C4 to C123, C5 to C118, C7 to C125, C8 to C119, D1 to D102, D2 to D100, D3 to D101, IC1 to IC103, IC10 to IC106, IC2 to IC107, IC3 to IC102, IC4 to IC101, IC5 to IC109, IC6 to IC104, IC7 to IC108, IC8 to IC100, IC9 to IC105, OK1 to OK100, Q1 to Q101, Q2 to Q100, R1 to R104, R10 to R111, R11 to R129, R12 to R113, R13 to R107, R14 to R123, R15 to R126, R16 to R112, R17 to R156, R18 to R155, R19 to R158, R2 to R106, R20 to R161, R21 to R160, R22 to R162, R23 to R159, R24 to R157, R25 to R153, R26 to R105, R27 to R154, R28 to R119, R29 to R152, R3 to R137, R30 to R120, R31 to R132, R32 to R122, R33 to R131, R34 to R115, R35 to R127, R36 to R167, R37 to R166, R38 to R165, R39 to R168, R4 to R124, R40 to R164, R41 to R163, R42 to R102, R43 to R103, R44 to R128, R45 to R130, R46 to R114, R47 to R147, R48 to R148, R49 to R151, R5 to R117, R50 to R149, R51 to R146, R52 to R116, R53 to R121, R54 to R134, R55 to R133, R56 to R109, R57 to R150, R58 to R118, R59 to R125, R6 to R110, R60 to R100, R61 to R101, R7 to R136, R8 to R135, R9 to R108, U1 to U100
Connections:
- new net N$61: R136.A, R142.2
- new net N$62: R136.E, R143.2
- new net N$63: R135.A, R140.2
- new net N$65: R135.E, R141.2
- new net N$67: R134.A, R139.2
- new net N$68: R134.E, R138.2
- new net N$69: R133.A, R144.2
- new net N$70: R133.E, R145.2
- net +5V: now also C103.+; no longer C9.+
- net -5V_ACCURATE: now also R139.1, R140.1, R142.1, R144.1; no longer R133.A, R134.A, R135.A, R136.A
- net 5V_ACCURATE: now also R138.1, R141.1, R143.1, R145.1; no longer R133.E, R134.E, R135.E, R136.E
- net DAC_TONE: now also C107.+; no longer C6.+
- net GND: now also C100.-, C103.-, C109.+, J100.3, J100.4, J100.5, J100.6, J100.7, J100.8, J7.1; no longer C10.+, C12.-, C9.-, J11.1, J7.3, J7.4, J7.5, J7.6, J7.7, J7.8
- net N$11: now also J5.3; no longer J1.3
- net N$14: now also J6.3; no longer J2.3
- net N$16: now also J2.3; no longer J8.3
- net N$17: now also C107.-; no longer C6.-
- net N$18: now also J1.3; no longer J6.3
- net N$26: now also J7.3; no longer J3.3
- net N$40: now also C128.-; no longer C24.-
- net N$53: now also J3.3; no longer J9.3
- net N$54: now also J4.3; no longer J11.3
- net N$56: now also J100.1, J100.2; no longer J7.1, J7.2
- net N$6: now also C128.+, J9.3; no longer C24.+, J5.3
- net N$64: now also J100.10, J100.9; no longer J7.10, J7.9
- net TONE_OUT: now also J8.3; no longer J4.3
- net VCC: now also C100.+; no longer C12.+
- net VEE: now also C109.-; no longer C10.-
Other:
- note added: "forestcaver 2020; original deisgn Émilie Gillet, 2012. cc-by-sa"
