File: AJH_LPG/lpg_v22_4hp.brd (EAGLE design)
At the start: 19 x 108.4 mm, 48 parts, among them IC1 DG212CJD, IC2 TL074D, J100 PJ301_THONKICONN6, J101 PJ301_THONKICONN6, J102 PJ301_THONKICONN6, SW100 submini-2T

Commit message: Updated footprint for vactrol on lpg
Connections:
- net N$45: now also V1.2; no longer V1.1
- net N$46: now also V1.1; no longer V1.2
Routing:
- net N$45: track 9.18 -> 11.7 mm
- net N$46: track 6.79 -> 8.96 mm
Other:
- board text added: "LPG v1.2 by forestcaver, copyright 2020"
- board text removed: "LPG v1.1 by forestcaver, copyright 2020"
Changed lines of the file:
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@@
 <?xml version="1.0" encoding="utf-8"?>
 <!DOCTYPE eagle SYSTEM "eagle.dtd">
-<eagle version="9.5.2">
+<eagle version="9.6.2">
 <drawing>
 <settings>
@@
 <wire x1="0" y1="108.43" x2="0" y2="0" width="0.1524" layer="20"/>
 <wire x1="2.8575" y1="107.6326" x2="2.8575" y2="101.2826" width="0.1524" layer="21"/>
-<text x="0.9525" y="39.0525" size="0.6096" layer="21" rot="R270">LPG v1.1 by forestcaver,
+<text x="0.9525" y="39.0525" size="0.6096" layer="21" rot="R270">LPG v1.2 by forestcaver,
 copyright 2020</text>
 <wire x1="0.3175" y1="107.6326" x2="0.3175" y2="101.2826" width="0.1524" layer="21"/>
@@
 <contactref element="R1" pad="2"/>
 <contactref element="D3" pad="A"/>
-<contactref element="V1" pad="1"/>
-<wire x1="3.175" y1="83.185" x2="1.5875" y2="84.7725" width="0.2032" layer="1"/>
-<wire x1="1.5875" y1="84.7725" x2="1.5875" y2="87.9525" width="0.2032" layer="1"/>
+<contactref element="V1" pad="2"/>
 <wire x1="3.175" y1="87.9475" x2="3.175" y2="89.965" width="0.2032" layer="1"/>
 <wire x1="3.175" y1="89.965" x2="3.2775" y2="90.0675" width="0.2032" layer="1"/>
 <wire x1="1.5875" y1="87.9525" x2="3.17" y2="87.9525" width="0.2032" layer="1"/>
 <wire x1="3.17" y1="87.9525" x2="3.175" y2="87.9475" width="0.2032" layer="1"/>
+<wire x1="1.5875" y1="87.9525" x2="1.5875" y2="82.2325" width="0.2032" layer="1"/>
+<wire x1="1.5875" y1="82.2325" x2="3.175" y2="80.645" width="0.2032" layer="1"/>
 </signal>
 <signal name="N$46">
-<contactref element="V1" pad="2"/>
+<contactref element="V1" pad="1"/>
 <contactref element="R3" pad="2"/>
-<wire x1="7.9375" y1="76.2" x2="7.9375" y2="76.5175" width="0.2032" layer="1"/>
-<wire x1="7.9375" y1="76.5175" x2="3.81" y2="80.645" width="0.2032" layer="1"/>
-<wire x1="3.81" y1="80.645" x2="3.175" y2="80.645" width="0.2032" layer="1"/>
+<wire x1="3.175" y1="83.185" x2="7.9375" y2="78.4225" width="0.2032" layer="1"/>
+<wire x1="7.9375" y1="78.4225" x2="7.9375" y2="76.2" width="0.2032" layer="1"/>
 </signal>
 <signal name="N$47">
