File: AJH_LPG/lpg_v22_4hp.sch (EAGLE design)
At the start: 48 parts, among them IC1 DG212CJD, IC2 TL074D, J100 PJ301_THONKICONN6, J101 PJ301_THONKICONN6, J102 PJ301_THONKICONN6, SW100 submini-2T

Commit message: Updated footprint for vactrol on lpg
Changed lines of the file:
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@@
 <?xml version="1.0" encoding="utf-8"?>
 <!DOCTYPE eagle SYSTEM "eagle.dtd">
-<eagle version="9.5.2">
+<eagle version="9.6.2">
 <drawing>
 <settings>
