File: AJH_2B_VCA/AJH_2b_v1_03.brd (EAGLE design)
At the start: 20 x 108.4 mm, 118 parts, among them IC1 LM4040B10, IC2 LM4040B10, IC3 V2164SZ, IC4 V2164SZ, IC5 OPA4171, IC6 OPA4171, IC7 OPA4171, IC8 OPA4171, J100 PJ301_THONKICONN6, J101 PJ301_THONKICONN6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

Commit message: Update README.md
Update 2B

error
Parts:
- removed C8, C9: 100n, rcl:C0402
- removed IC4: V2164SZ, ssm2164:SOIC16N
- removed R4: DNP, resistor:R0402
- moved C12 7.46 mm to (15.9, 81.2)
- moved R5 6.83 mm to (3.96, 87.3), turned to 0 degrees
- moved IC3 5.31 mm to (9.96, 82.8)
- moved R6 4.60 mm to (15.9, 80.0), turned to 180 degrees
- moved C7 2.72 mm to (16.1, 87.3)
- moved C10 2.66 mm to (15.8, 78.5), turned to 180 degrees
- moved J1 2.50 mm to (2.52, 38.0), turned to 270 degrees
- moved R45 0.32 mm to (7.72, 23.1)
Connections:
- removed net N$86: IC4.1, R4.2
- net FOO2: now also IC3.2; no longer IC4.2
- net GND: no longer C8.2, C9.1, IC4.8
- net N$46: now also IC3.15; no longer IC4.15
- net N$48: now also IC3.13; no longer IC4.13
- net N$67: now also IC3.4; no longer IC4.4
- net N$68: now also IC3.14, IC3.3; no longer IC4.14, IC4.3
- net VCC: no longer C8.1, IC4.16, R4.1
- net VEE: no longer C9.2, IC4.9
Routing:
- net VEE: track 147.7 -> 123.0 mm, vias 9 -> 6
- net AREF_+10: track 124.1 -> 117.8 mm
- net N$48: track 70.7 -> 75.9 mm
- net N$24: track 33.6 -> 38.6 mm
- net FOO2: track 11.8 -> 16.8 mm
- net OUT: track 14.8 -> 19.5 mm
- net N$86: track 4.53 -> 0.00 mm
- net N$26: track 57.5 -> 61.3 mm
- net N$31: track 57.7 -> 54.0 mm, vias 2 -> 1
- net N$46: track 48.7 -> 52.0 mm
- net VCC: track 131.7 -> 129.7 mm
- net N$34: track 21.2 -> 19.2 mm
- net N$43: track 26.6 -> 24.7 mm
- net N$68: track 37.3 -> 39.0 mm
- net N$67: track 80.3 -> 81.6 mm
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Other:
- board text added: "2B v1.03 copyright forestcaver 2020"
- board text added: "GND"
- board text added: "In"
- board text added: "OUT"
- board text added: "Out"
- board text removed: "2B v1.01 copyright forestcaver 2020"
