File: AJH_2B_VCA/AJH_2b_v1_03.sch (EAGLE design)
At the start: 118 parts, among them IC1 LM4040B10, IC2 LM4040B10, IC3 V2164SZ, IC4 V2164SZ, IC5 OPA4171, IC6 OPA4171, IC7 OPA4171, IC8 OPA4171, J100 PJ301_THONKICONN6, J101 PJ301_THONKICONN6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

Commit message: Update README.md
Update 2B

error
Parts:
- removed C8, C9: 100n, rcl:C-USC0402
- removed IC4: V2164SZ, ssm2164:SSM2164S
- removed R4: DNP, resistor:R-US_R0402
Connections:
- removed net N$86: IC4E.MODE, R4.2
- net FOO2: now also IC3A.IN; no longer IC4A.IN
- net GND: no longer C8.2, C9.1, IC4E.GND
- net N$46: now also IC3D.IN; no longer IC4D.IN
- net N$48: now also IC3D.OUT; no longer IC4D.OUT
- net N$67: now also IC3A.OUT; no longer IC4A.OUT
- net N$68: now also IC3A.CTRL, IC3D.CTRL; no longer IC4A.CTRL, IC4D.CTRL
- net VCC: no longer C8.1, IC4E.V+, R4.1
- net VEE: no longer C9.2, IC4E.V-
